File: Hardware/Buck_Converter/Buck_Converter.kicad_sch (KiCad schematic)
At the start: 17 parts, among them J1 Conn_01x05, U1 AP62200WU, U2 AP62200WU

Commit message: Prepare for board review
Other:
- company: MRDT -> Mars Rover Design Team
Changed lines of the file:
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@@
 		(date "2025-04-01")
 		(rev "1")
-		(company "MRDT")
+		(company "Mars Rover Design Team")
 		(comment 1 "Brendan Westley")
+		(comment 2 "Malacki Ehlers")
 	)
 	(junction
