File: Hardware/board/Smart_MoCo.kicad_sch (KiCad schematic)
At the start: 35 parts, among them J1 Conn_01x02, J2 Conn_01x04, J3 Conn_01x02, J4 Conn_01x02, J5 Conn_01x04, J6 1722861102, J7 1722861102, U1 STM32F042F6Px, U2 VNH5019A-E, U3 SN65HVD232, U4 AP62200WU

Commit message: Redesign hardware
Parts:
- removed D1: Red, LED_SMD:LED_0603_1608Metric_Pad1.05x0.95mm_HandSolder, symbol Device:LED
- removed J4: Conn_01x02, Connector_JST:JST_SH_SM02B-SRSS-TB_1x02-1MP_P1.00mm_Horizontal, symbol Connector_Generic:Conn_01x02
- removed J6, J7: 1722861102, MRDT_Connectors:CONN_SD-172286-1000_02_MOL, symbol MRDT_Connectors:1722861102
- added C4, C5: 22uF, Capacitor_SMD:C_0603_1608Metric_Pad1.08x0.95mm_HandSolder, symbol Device:C
- added D1: LED_RGBK, Smart_MoCo:PLCC4_3p5x2p8_SLD-L, symbol Device:LED_RGBK
- added J5, J6: 1723103102, MRDT_Connectors:CONN_1723102000_02_MOL, symbol MRDT_Connectors:1723103102
- added R10, R9: 1k, Resistor_SMD:R_0603_1608Metric_Pad0.98x0.95mm_HandSolder, symbol Device:R
- H1, H2: footprint Local Libraries:Minimal_4_40_Hole -> Smart_MoCo:Minimal_4_40_Hole
- J1, J3: footprint Connector_JST:JST_SH_SM02B-SRSS-TB_1x02-1MP_P1.00mm_Horizontal -> Connector_JST:JST_XH_S2B-XH-A_1x02_P2.50mm_Horizontal
- J2: footprint Connector_JST:JST_SH_SM04B-SRSS-TB_1x04-1MP_P1.00mm_Horizontal -> Connector_JST:JST_XH_S4B-XH-A_1x04_P2.50mm_Horizontal
- renumbered C8 to C10, C5 to C7, C4 to C8, C7 to C9, J5 to J4, R10 to R11, R9 to R12
Connections:
- net +12V: now also J5.1
- net +3V3: now also C4.1, C5.1; no longer J3.1 (Pin_1)
- net GND: now also C4.2, C5.2, D1.4 (K), J5.2
- net LIM_A: now also J3.1 (Pin_1); no longer J3.2 (Pin_2)
- net LIM_B: now also J3.2 (Pin_2)
- net OUTA: now also J6.1
- net OUTB: now also J6.2
- net at R8.2: now also D1.1 (RA)
- net LED_R: now reaches U1.12 (PA6)
- net LED_R: now also R8.1
- net LED_G: now reaches U1.3 (PF1)
- net LED_G: now also R9.1
- net LED_STATUS renamed LED_B
- net LED_B: now also R10.1; no longer R8.1
- new net: D1.2 (GA), R9.2
- new net: D1.3 (BA), R10.2
- no-connect marks 5 -> 3
Other:
- note added: "See driver datasheet figure 4 1k resistors in series with input pins were removed and VBAT and VCC are shorted as reverse battery protection is not implemented"
- note removed: "See driver datasheet figure 4 1k resistors in series with input pins may be removed and VBAT and VCC are shorted as reverse battery protection is not implemented"
- moved on the sheet: C1, D2, D3, R1, R11, R12, R2, R3, R4, U2

Commit message: Incorporate review 1 feedback
Parts:
- removed J5, J6: 1723103102, MRDT_Connectors:CONN_1723102000_02_MOL, symbol MRDT_Connectors:1723103102
- added C11: 100nF, Capacitor_SMD:C_0603_1608Metric_Pad1.08x0.95mm_HandSolder, symbol Device:C
- added D4: MMSZ5240BT1G, MRDT_Devices:SOD-123_ONS-L, symbol MRDT_Devices:MMSZ5240BT1G
- added J5, J6: Molex_UltraFit_02, MRDT_Connectors:CONN_1723102000_02_MOL, symbol MRDT_Connectors:Molex_UltraFit_02
- added J7: Conn_01x01, Connector_Wire:SolderWire-0.5sqmm_1x01_D0.9mm_OD2.1mm, symbol Connector_Generic:Conn_01x01
- added R13: 10k, Resistor_SMD:R_0603_1608Metric_Pad0.98x0.95mm_HandSolder, symbol Device:R
- added U5: TPC8132_LQS, Package_SO:SOIC-8_3.9x4.9mm_P1.27mm, symbol MRDT_Devices:TPC8132_LQS
Connections:
- net +12V: now also D4.1, U5.1 (S), U5.2, U5.3
- net +3V3: now also C11.1
- net GND: now also C11.2, J5.2, R13.2; no longer U1.1 (PB8)
- net IN_A: now also U1.3 (PF1); no longer U1.14 (PB1)
- net IN_B: now also U1.2 (PF0); no longer U1.13 (PA7)
- net LED_B: now also U1.14 (PB1); no longer U1.2 (PF0)
- net LED_G: now also U1.13 (PA7); no longer U1.3 (PF1)
- net OUTA: now also J6.1
- net OUTB: now also J6.2
- new net: D4.2, R13.1, U5.4 (G)
- new net: J5.1, U5.5 (D), U5.6, U5.7, U5.8
- new net GPIO: J7.1 (Pin_1), U1.1 (PB8)
Other:
- note removed: "PB8-BOOT0 tied low to disable system bootloader; see AN2606"
- moved on the sheet: C2, C3, C4, C5, J3, L1, R6, R7, U4

Commit message: Incorporate review 2 feedback
Parts:
- removed J5, J6: Molex_UltraFit_02, MRDT_Connectors:CONN_1723102000_02_MOL, symbol MRDT_Connectors:Molex_UltraFit_02
- added J5, J6: Molex_UltraFit_02_Horizontal, MRDT_Connectors:MOLEX_UltraFit_02_Horizontal, symbol MRDT_Connectors:Molex_UltraFit_02_Horizontal
Connections:
- net GND: now also J5.2, J5.MP, J6.MP
- net OUTA: now also J6.1
- net OUTB: now also J6.2
- net at U5.5 (D), U5.6, U5.7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: now also J5.1
