File: Hardware/SMoCo_board/smoco.kicad_sch (KiCad schematic)
At the start: 0 parts

Commit message: Testing local symbol import
Parts:
- added U1: VNH7040AYTR, POWERSSO-36TP_STM, symbol VNH7040AYTR:VNH7040AYTR
Connections:
- no-connect marks 0 -> 1
Changed lines of the file:
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@@
 	(generator_version "10.0")
 	(paper "A4")
+	(no_connect
+		(at 55.88 55.88)
+	)
+	(symbol
+		(lib_id "VNH7040AYTR:VNH7040AYTR")
+		(at 105.41 72.39 0)
+		(unit 1)
+		(body_style 1)
+		(exclude_from_sim no)
+		(in_bom yes)
+		(on_board yes)
+		(in_pos_files yes)
+		(dnp no)
+		(fields_autoplaced yes)
+		(property "Reference" "U1"
+			(at 125.73 62.23 0)
+			(show_name no)
+			(do_not_autoplace no)
+			(effects
+				(font
+					(size 1.524 1.524)
+				)
+			)
+		)
+		(property "Value" "VNH7040AYTR"
+			(at 125.73 64.77 0)
+			(show_name no)
+			(do_not_autoplace no)
+			(effects
+				(font
+					(size 1.524 1.524)
+				)
+			)
+		)
+		(property "Footprint" "POWERSSO-36TP_STM"
+			(at 105.41 72.39 0)
+			(hide yes)
+			(show_name no)
+			(do_not_autoplace no)
+			(effects
+				(font
+					(size 1.27 1.27)
+					(italic yes)
+				)
+			)
+		)
+		(property "Datasheet" "https://www.st.com/resource/en/datasheet/vnh7040ay.pdf"
+			(at 105.41 72.39 0)
+			(hide yes)
+			(show_name no)
+			(do_not_autoplace no)
+			(effects
+				(font
+					(size 1.27 1.27)
+					(italic yes)
+				)
+			)
+		)
+		(property "Description" ""
+			(at 105.41 72.39 0)
+			(hide yes)
+			(show_name no)
+			(do_not_autoplace no)
+			(effects
+				(font
+					(size 1.27 1.27)
+				)
+			)
+		)
+		(pin "16"
+		)
+		(pin "20"
+		)
+		(pin "22"
+		)
+		(pin "25"
+		)
+		(pin "28"
+		)
+		(pin "8"
+		)
+		(pin "6"
+		)
+		(pin "23"
+		)
+		(pin "1"
+		)
+		(pin "13"
+		)
+		(pin "27"
+		)
+		(pin "4"
+		)
+		(pin "9"
+		)
+		(pin "2"
+		)
+		(pin "3"
+		)
+		(pin "10"
+		)
+		(pin "11"
+		)
+		(pin "7"
+		)
+		(pin "5"
+		)
+		(pin "12"
+		)
+		(pin "14"
+		)
+		(pin "15"
+		)
+		(pin "17"
+		)
+		(pin "18"
+		)
+		(pin "19"
+		)
+		(pin "21"
+		)
+		(pin "24"
+		)
+		(pin "26"
+		)
+		(pin "31"
+		)
+		(pin "32"
+		)
+		(pin "39"
+		)
+		(pin "37"
+		)
+		(pin "29"
+		)
+		(pin "35"
+		)
+		(pin "33"
+		)
+		(pin "36"
+		)
+		(pin "38"
+		)
+		(pin "30"
+		)
+		(pin "34"
+		)
+		(instances
+			(project "smoco"
+				(path "/e05f0fda-5136-4f92-92b6-924779ff6aac"
+					(reference "U1")
+					(unit 1)
+				)
+			)
+		)
+	)
 	(sheet_instances
 		(path "/"
