File: Hardware/SMoCo_board/SMoCo_board.kicad_sch (KiCad schematic)
At the start: 0 parts

Commit message: hi
Parts:
- added C1, C4: 100nF, symbol Device:C
- added C2: 470nF, symbol Device:C
- added C3, C5: C, symbol Device:C
- added C6: 10uF, symbol Device:C
- added D1: D_Zener, symbol Device:D_Zener
- added D2, D3, D4: LED, symbol Device:LED
- added J1, J2, J3, J4, J6, J8: Conn_01x02, symbol Connector_Generic:Conn_01x02
- added J5: Conn_01x06, symbol Connector_Generic:Conn_01x06
- added J7: Conn_01x04, symbol Connector_Generic:Conn_01x04
- added L1: L, symbol Device:L
- added Q1: Q_PMOS, symbol Device:Q_PMOS
- added R1, R2, R3, R4, R5, R6, R7, R8: 1k, symbol Device:R_US
- added R10: 5.5k, symbol Device:R_US
- added R11, R13: 330, symbol Device:R_US
- added R12: 120, symbol Device:R_US
- added R9: Rsense, symbol Device:R_US
- added U1: STM32F072C8T6, LQFP48-7x7mm, symbol STM32F072C8T6:STM32F072C8T6
- added U2: VNH7040AYTR, POWERSSO-36TP_STM, symbol VNH7040AYTR:VNH7040AYTR
- added U3: SN65HVD232, Package_SO:SOIC-8_3.9x4.9mm_P1.27mm, symbol Interface_CAN_LIN:SN65HVD232
- added U4: AP63203WU, Package_TO_SOT_SMD:TSOT-23-6, symbol Regulator_Switching:AP63203WU
Connections:
- new net: D4.2 (A), R13.2
- new net: C4.1, U4.5 (SW)
- new net: C4.2, L1.1, U4.6 (BST)
- new net: D3.2 (A), R11.2
- new net: D2.2 (A), R10.2
- new net: D1.2 (A), Q1.G, R1.1
- new net +24V: C1.1, C2.1, C6.1, D1.1 (K), Q1.S, R10.1, U2.10 (Vcc), U2.27 (Vcc), U4.2 (EN), U4.3 (IN)
- new net +3.3V: C5.1, J5.6 (Pin_6), J7.1 (Pin_1), L1.2, R11.1, U1.1 (VBAT), U1.24 (VDD), U1.36 (VDDIO2), U1.48 (VDD), U1.9 (VDDA), U3.3 (VCC), U4.1 (FB)
- new net ABS: J5.5 (Pin_5), U1.38 (PA15)
- new net CAN RX: U1.32 (PA11), U3.4 (R)
- new net CAN TX: U1.33 (PA12), U3.1 (D)
- new net CANH: J6.2 (Pin_2), J8.2 (Pin_2), R12.1, U3.7 (CANH)
- new net CANL: J6.1 (Pin_1), J8.1 (Pin_1), R12.2, U3.6 (CANL)
- new net ENC A: J5.4 (Pin_4), U1.18 (PB0)
- new net ENC B: J5.3 (Pin_3), U1.19 (PB1)
- new net ENC I: J5.2 (Pin_2), U1.20 (PB2)
- new net GND: C1.2, C2.2, C3.2, C5.2, C6.2, D2.1 (K), D3.1 (K), D4.1 (K), J2.1 (Pin_1), J5.1 (Pin_1), J7.4 (Pin_4), R1.2, R9.2, U1.23 (VSS), U1.35 (VSS), U1.47 (VSS), U1.8 (VSSA), U2.3 (GND_A), U2.30 (GND_B), U2.31 (GND_B), U2.32 (GND_B), U2.33 (GND_B), U2.34 (GND_B), U2.4 (GND_A), U2.5 (GND_A), U2.6 (GND_A), U2.7 (GND_A), U3.2 (GND), U4.4 (GND)
- new net IN_A IN: R2.1, U2.16 (IN_A)
- new net IN_A OUT: R2.2, U1.10 (PA0)
- new net IN_B IN: R3.1, U2.21 (IN_B)
- new net IN_B OUT: R3.2, U1.11 (PA1)
- new net LIM1 A: J3.1 (Pin_1), U1.29 (PA8)
- new net LIM1 B: J3.2 (Pin_2), U1.30 (PA9)
- new net LIM2 A: J4.1 (Pin_1), U1.39 (PB3)
- new net LIM2 B: J4.2 (Pin_2), U1.40 (PB4)
- new net MOTOR PWR A: J1.1 (Pin_1), U2.11 (Source_HSD_A), U2.12 (Source_HSD_A), U2.13 (Source_HSD_A), U2.14 (Source_HSD_A), U2.2 (Drain_LSD_A), U2.8 (Drain_LSD_A), U2.9 (Drain_LSD_A)
- new net MOTOR PWR B: J1.2 (Pin_2), U2.23 (Source_HSD_B), U2.24 (Source_HSD_B), U2.25 (Source_HSD_B), U2.26 (Source_HSD_B), U2.28 (Drain_LSD_B), U2.29 (Drain_LSD_B), U2.35 (Drain_LSD_B)
- new net MS IN: R7.2, R9.1, U1.15 (PA5)
- new net MS OUT: C3.1, R7.1, U2.19 (MultiSense)
- new net MS_EN IN: R8.1, U2.20 (MultiSense_EN)
- new net MS_EN OUT: R8.2, U1.14 (PA4)
- new net Motor LED: R13.1, U1.41 (PB5)
- new net PWM IN: R4.1, U2.17 (PWM)
- new net PWM OUT: R4.2, U1.17 (PA7)
- new net SEL0 IN: R5.1, U2.15 (SEL0)
- new net SEL0 OUT: R5.2, U1.12 (PA2)
- new net SEL1 IN: R6.1, U2.22 (SEL1)
- new net SEL1 OUT: R6.2, U1.13 (PA3)
- new net SWDCLK: J7.2 (Pin_2), U1.37 (PA14)
- new net SWDIO: J7.3 (Pin_3), U1.34 (PA13)
- new net Vaux: J2.2 (Pin_2), Q1.D
- no-connect marks 0 -> 6

Commit message: fix bug
this was gavin lmao
Parts:
- added C7: 100nF, symbol Device:C
- added D?: LED, symbol Device:LED
- added R?: 330, symbol Device:R_US
Connections:
- net +3.3V: now also C7.1
- net GND: now also C7.2, D?.1 (K)
- net IN_A OUT: now also R13.1
- net IN_B OUT: now also R?.1
- net Motor LED: no longer names the net of U1.41 (PB5)
- net Motor LED: no longer R13.1
- new net: D?.2 (A), R?.2
Other:
- note added: "24v LED"
- note added: "3.3v LED"
- note added: "BUCK CONVERTER"
- note added: "CAN CONNECTORS"
- note added: "CAN TRANSCIEVER"
- note added: "CONNECTORS"
- note added: "ENCODER"
- note added: "LED"
- note added: "LIMIT SWITCH"
- note added: "MICROCONTROLLER CORE"
- note added: "MOTOR DRIVER"
- note added: "MOTOR PLUG IN"
- note added: "Motor Activity"
- note added: "POWER"
- note added: "REVERSE VOLTAGE PROTECTION"
- note added: "SWD"
- moved on the sheet: C1, C2, C3, C4, C5, C6, D1, D2, D3, D4, J1, J2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
