File: Hardware/SMoCo_board/SMoCo_board.kicad_sch (KiCad schematic)
At the start: 46 parts, among them J1 Conn_01x02, J2 Conn_01x02, J3 Conn_01x02, J4 Conn_01x02, J5 Conn_01x06, J6 Conn_01x02, J7 Conn_01x04, J8 Conn_01x02, Q1 Q_PMOS, U1 STM32F072C8T6, U2 VNH7040AYTR, U3 SN65HVD232, U4 AP63203WU

Commit message: smoco
Pin rework
Parts:
- removed J3: Conn_01x02, symbol Connector_Generic:Conn_01x02
- gave numbers to parts that had none: 8
Connections:
- net ABS: no longer J5.5 (Pin_5)
- net ENC I: now also U1.28 (PB15)
- net LED_B: now also U1.46 (PB9); no longer U1.43 (PB7)
- net LED_G: now also U1.45 (PB8); no longer U1.42 (PB6)
- net LIM2 A: no longer J4.1 (Pin_1)
- net LIM2 B: no longer J4.2 (Pin_2)
- net ENC ABS: now reaches U1.27 (PB14)
- net ENC ABS: now also J5.5 (Pin_5)
- net ENC_B: now reaches U1.31 (PA10)
- net LIM1 A: no longer names the net of U1.29 (PA8)
- net LIM1 B renamed ENC_A
- new net LIM A: J4.1 (Pin_1), U1.42 (PB6)
- new net LIM B: J4.2 (Pin_2), U1.43 (PB7)
Other:
- moved on the sheet: D2, D3, D4, D6, LED1, R10, R11, R13, R14, R15, R16, R17

Commit message: Smoco
Parts:
- added D?: D_Zener, Diode_THT:D_DO-41_SOD81_P10.16mm_Horizontal, symbol Device:D_Zener
- added H1: MountingHole, SX1262IMLTRT:QFN50P400X400X100-25N, symbol Mechanical:MountingHole
- added H2: MountingHole, symbol Mechanical:MountingHole
Other:
- note added: "Mounting Holes"

Commit message: smoco
 temp update
Parts:
- removed D5: >=3v3, Package_SON:WSON-6-1EP_2x2mm_P0.65mm_EP1x1.6mm, symbol Device:D_TVS
- gave numbers to parts that had none: 1
Connections:
- net +3.3V: now also D2.1 (K)
- net GND: now also D2.2 (A)
Other:
- moved on the sheet: D2
Changed lines of the file:
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@@
 	)
 	(junction
-		(at 147.32 20.32)
-		(diameter 0)
-		(color 0 0 0 0)
-	)
-	(junction
 		(at 147.32 30.48)
 		(diameter 0)
@@
 	)
 	(junction
+		(at 147.32 20.32)
+		(diameter 0)
+		(color 0 0 0 0)
+	)
+	(junction
 		(at 147.32 31.75)
 		(diameter 0)
@@
 	(wire
 		(pts
-			(xy 147.32 20.32) (xy 147.32 27.94)
+			(xy 147.32 19.05) (xy 147.32 20.32)
 		)
 		(stroke
@@
 	(wire
 		(pts
-			(xy 92.71 40.64) (xy 92.71 38.1)
-		)
-		(stroke
-			(width 0)
-			(type default)
-		)
-	)
-	(wire
-		(pts
 			(xy 46.99 26.67) (xy 46.99 24.13)
 		)
@@
 	(wire
 		(pts
+			(xy 147.32 20.32) (xy 147.32 27.94)
+		)
+		(stroke
+			(width 0)
+			(type default)
+		)
+	)
+	(wire
+		(pts
 			(xy 265.43 134.62) (xy 275.59 134.62)
 		)
@@
 	(wire
 		(pts
-			(xy 90.17 40.64) (xy 90.17 41.91)
+			(xy 92.71 38.1) (xy 92.71 41.91)
 		)
 		(stroke
@@
 	(wire
 		(pts
-			(xy 90.17 41.91) (xy 151.13 41.91)
+			(xy 92.71 41.91) (xy 151.13 41.91)
 		)
 		(stroke
@@
 	(wire
 		(pts
-			(xy 90.17 40.64) (xy 92.71 40.64)
-		)
-		(stroke
-			(width 0)
-			(type default)
-		)
-	)
-	(wire
-		(pts
 			(xy 222.25 104.14) (xy 213.36 104.14)
 		)
@@
 	(wire
 		(pts
-			(xy 147.32 19.05) (xy 147.32 20.32)
-		)
-		(stroke
-			(width 0)
-			(type default)
-		)
-	)
-	(wire
-		(pts
 			(xy 34.29 83.82) (xy 58.42 83.82)
 		)
@@
 	)
 	(symbol
-		(lib_id "Device:D_TVS")
-		(at 151.13 20.32 180)
-		(unit 1)
-		(body_style 1)
-		(exclude_from_sim no)
-		(in_bom yes)
-		(on_board yes)
-		(in_pos_files yes)
-		(dnp no)
-		(fields_autoplaced yes)
-		(property "Reference" "D5"
-			(at 151.13 13.97 0)
-			(show_name no)
-			(do_not_autoplace no)
-			(effects
-				(font
-					(size 1.27 1.27)
-				)
-			)
-		)
-		(property "Value" ">=3v3"
-			(at 151.13 16.51 0)
-			(show_name no)
-			(do_not_autoplace no)
-			(effects
-				(font
-					(size 1.27 1.27)
-				)
-			)
-		)
-		(property "Footprint" "Package_SON:WSON-6-1EP_2x2mm_P0.65mm_EP1x1.6mm"
-			(at 151.13 20.32 0)
-			(hide yes)
-			(show_name no)
-			(do_not_autoplace no)
-			(effects
-				(font
-					(size 1.27 1.27)
-				)
-			)
-		)
-		(property "Datasheet" ""
-			(at 151.13 20.32 0)
-			(hide yes)
-			(show_name no)
-			(do_not_autoplace no)
-			(effects
-				(font
-					(size 1.27 1.27)
-				)
-			)
-		)
-		(property "Description" "Bidirectional transient-voltage-suppression diode"
-			(at 151.13 20.32 0)
-			(hide yes)
-			(show_name no)
-			(do_not_autoplace no)
-			(effects
-				(font
-					(size 1.27 1.27)
-				)
-			)
-		)
-		(pin "1"
-		)
-		(pin "2"
-		)
-		(instances
-			(project "SMoCo_board"
-				(path "/ad6ab0ba-09d2-4577-bf28-b79b9df619ef"
-					(reference "D5")
-					(unit 1)
-				)
-			)
-		)
-	)
-	(symbol
 		(lib_id "power:GND")
 		(at 19.05 34.29 0)
@@
 	(symbol
 		(lib_id "Device:D_Zener")
-		(at 139.7 17.78 0)
+		(at 151.13 20.32 0)
 		(unit 1)
 		(body_style 1)
@@
 		(dnp no)
 		(fields_autoplaced yes)
-		(property "Reference" "D?"
-			(at 139.7 11.43 0)
+		(property "Reference" "D2"
+			(at 151.13 13.97 0)
 			(show_name no)
 			(do_not_autoplace no)
@@
 		)
 		(property "Value" "D_Zener"
-			(at 139.7 13.97 0)
+			(at 151.13 16.51 0)
 			(show_name no)
 			(do_not_autoplace no)
@@
 		)
 		(property "Footprint" "Diode_THT:D_DO-41_SOD81_P10.16mm_Horizontal"
-			(at 139.7 17.78 0)
+			(at 151.13 20.32 0)
 			(hide yes)
 			(show_name no)
@@
 			)
 		)
-		(property "Datasheet" ""
-			(at 139.7 17.78 0)
+		(property "Datasheet" "https://www.panjit.com.tw/upload/datasheet/BZX584C2V4_SERIES.pdf"
+			(at 151.13 20.32 0)
 			(hide yes)
 			(show_name no)
@@
 		)
 		(property "Description" "Zener diode"
-			(at 139.7 17.78 0)
+			(at 151.13 20.32 0)
 			(hide yes)
 			(show_name no)
@@
 			(project "SMoCo_board"
 				(path "/ad6ab0ba-09d2-4577-bf28-b79b9df619ef"
-					(reference "D?")
+					(reference "D2")
 					(unit 1)
 				)

Commit message: SmoCo
update
Parts:
- removed C1: 100nF, symbol Device:C
- removed C2: 470nF, symbol Device:C
- removed D1: 15V, symbol Device:D_Zener
- removed Q1: Q_PMOS, symbol Device:Q_PMOS
- removed R1: 1k, symbol Device:R_US
- added C?: 100uf, Capacitor_SMD:C_0603_1608Metric_Pad1.08x0.95mm_HandSolder, symbol Device:C_Polarized
- added D3: MMSZ5240BT1G, MRDT_Devices:SOD-123_ONS-L, symbol MRDT_Devices:MMSZ5240BT1G
- added MOSFET1: TPC8132_LQS, MRDT_Devices:SOP-8_TOS-L, symbol MRDT_Devices:TPC8132_LQS
- added R3: 1k, Resistor_SMD:R_0603_1608Metric_Pad0.98x0.95mm_HandSolder, symbol Device:R_US
Connections:
- net +24V: now also D3.1, MOSFET1.1 (S), MOSFET1.2, MOSFET1.3
- net GND: now also C?.2, R3.2
- net Vaux: now also C?.1, MOSFET1.5 (D), MOSFET1.6, MOSFET1.7, MOSFET1.8
- new net: D3.2, MOSFET1.4 (G), R3.1
Other:
- moved on the sheet: H1, H2
