File: Hardware/SMoCo_board/Mosfet Circuit for RGB LED.kicad_sch (KiCad schematic)
At the start: 18 parts, among them Q1 BSS138, Q2 AO3401A, Q3 BSS138, Q4 AO3401A, Q5 BSS138, Q6 AO3401A

Commit message: Fixed lots of stuff
fixed LED resistor values, bulk capacitor, decoupling capacitors and most data sheets.
Parts:
- R15: value 200 -> 820
- R18: value 350 -> 820
- R21: value 1k -> 510
Changed lines of the file:
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@@
 			)
 		)
-		(property "Value" "1k"
+		(property "Value" "510"
 			(at 191.77 82.5499 0)
 			(show_name no)
@@
 			)
 		)
-		(property "Value" "200"
+		(property "Value" "820"
 			(at 105.41 82.5499 0)
 			(show_name no)
@@
 			)
 		)
-		(property "Value" "350"
+		(property "Value" "820"
 			(at 148.59 82.5499 0)
 			(show_name no)

Commit message: MS Resistor
Parts:
- removed Q1, Q3, Q5: BSS138, Package_TO_SOT_SMD:SOT-23, symbol Transistor_FET:BSS138
- removed Q2, Q4, Q6: AO3401A, Package_TO_SOT_SMD:SOT-23, symbol Transistor_FET:AO3401A
- removed R13, R16, R19: 5k, symbol Device:R_US
- removed R14, R17, R20: 10k, Resistor_THT:R_Array_SIP4, symbol Device:R_US
- removed R15, R18: 820, Resistor_THT:R_Array_SIP4, symbol Device:R_US
- removed R21: 510, Resistor_THT:R_Array_SIP4, symbol Device:R_US
- removed R22, R23, R24: 1k, Resistor_THT:R_Array_SIP4, symbol Device:R_US

Commit message: Fixed bug with MOSFET Hierarchal sheet
Parts:
- added Q1, Q3, Q5: BSS138, Package_TO_SOT_SMD:SOT-23, symbol Transistor_FET:BSS138
- added Q2, Q4, Q6: AO3401A, Package_TO_SOT_SMD:SOT-23, symbol Transistor_FET:AO3401A
- added R13, R16, R19: 5k, symbol Device:R_US
- added R14, R17, R20: 10k, Resistor_THT:R_Array_SIP4, symbol Device:R_US
- added R15: 200, Resistor_THT:R_Array_SIP4, symbol Device:R_US
- added R18: 350, Resistor_THT:R_Array_SIP4, symbol Device:R_US
- added R21, R22, R23, R24: 1k, Resistor_THT:R_Array_SIP4, symbol Device:R_US
Connections:
- new net: Q6.2 (S), R21.1
- new net: Q1.3 (D), R14.2
- new net: Q2.1 (G), R13.2, R14.1
- new net: Q2.2 (S), R15.1
- new net: Q6.1 (G), R19.2, R20.1
- new net: Q5.3 (D), R20.2
- new net: Q4.1 (G), R16.2, R17.1
- new net: Q3.3 (D), R17.2
- new net: Q4.2 (S), R18.1
- new net +24V: Q2.3 (D), Q4.3 (D), Q6.3 (D), R13.1, R16.1, R19.1
- new net GND: Q1.2 (S), Q3.2 (S), Q5.2 (S), R22.2, R23.2, R24.2
- new net LED_B: Q1.1 (G), R22.1
- new net LED_G: Q3.1 (G), R23.1
- new net LED_R: Q5.1 (G), R24.1
- new net Led_B_Out: R15.2
- new net Led_G_Out: R18.2
- new net Led_R_Out: R21.2
