File: Hardware/SMoCo_board/_restore_backup_2026-10-08T00-20-32-785/SMoCo_board.kicad_sch (KiCad schematic)
At the start: 46 parts, among them J1 Conn_01x02, J2 Conn_01x02, J3 Conn_01x02, J4 Conn_01x02, J5 Conn_01x06, J6 Conn_01x02, J7 Conn_01x04, J8 Conn_01x02, Q1 Q_PMOS, U1 STM32F072C8T6, U2 VNH7040AYTR, U3 SN65HVD232, U4 AP63203WU

Commit message: smoco
Recent Updated
Parts:
- removed C?: C, symbol Device:C
- removed D?: >=3v3, Package_SON:WSON-6-1EP_2x2mm_P0.65mm_EP1x1.6mm, symbol Device:D_TVS
- removed LED?: XZM2CRKM2DGFBB45SCCB, PLCC4_3p5x2p8_SLD, symbol 2026-10-08_05-14-25:XZM2CRKM2DGFBB45SCCB
- removed R?: 350, symbol Device:R_US
- removed R?: 200, symbol Device:R_US
- removed R?: 1k, symbol Device:R_US
- D1: value 15V -> D_Zener
- R13, R?: value 1k -> 330
Connections:
- net LED_B: no longer names the net of U1.43 (PB7)
- net LED_G: no longer names the net of U1.42 (PB6)
- net LED_R: no longer names the net of U1.41 (PB5)
Other:
- moved on the sheet: C5
